File: limbic_cm4/limbic_cm4.kicad_pcb (KiCad board)
At the start: 2 copper layers, 0 parts

Commit message: [New] Add rpi_cm4 to lib
Signed-off-by: Homalozoa <nx.tardis@gmail.com>
Parts:
- added U1: SC0320, Rolling_Custom:Raspberry-Pi-4-Compute-Module, F.Cu at (163.0, 100.0)
Other:
- board outline added: 92 x 52 mm
