File: limbic_cm4/limbic_cm4.kicad_sch (KiCad schematic)
At the start: 0 parts

Commit message: [New] Add rpi_cm4 to lib
Signed-off-by: Homalozoa <nx.tardis@gmail.com>
Parts:
- added U1: SC0320, Rolling_Custom:Raspberry-Pi-4-Compute-Module, symbol Rolling_Custom:SC0320
Connections:
- new net GND: U1.1 (GND), U1.107 (GND), U1.108 (GND), U1.113 (GND), U1.114 (GND), U1.119 (GND), U1.120 (GND), U1.125 (GND), U1.126 (GND), U1.13 (GND), U1.131 (GND), U1.132 (GND)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
