File: executor/executor.kicad_sch (KiCad schematic)
At the start: 135 parts, among them J1 XT30PW(2+2), Q1 WNM6006, Q2 WNM6006, Q3 WNM6006, Q4 WNM6006, Q5 WNM6006, Q6 WNM6006, U1 WD1601E, U2 DRV8323SRTAT, U3 GD32F303RETx, U4 TCAN4550RGYRQ1, U5 AS5047P-ATSM, U6 QMA7981, Y1 8M, Y2 40M

Commit message: [Modify] Change footprints for manufature
Signed-off-by: Homalozoa <nx.tardis@gmail.com>
Parts:
- C10, C6: value 10uF, 10%, 50V -> 10uF, 20%, 6.3V
- C16: value 100nF, 10%, 50V -> 100nF, 10%, 10V
- C17, C25, C29, C37, C65, C66: footprint Capacitor_SMD:C_0402_1005Metric -> Capacitor_SMD:C_0603_1608Metric
- C26, C28, C31, C34: footprint Capacitor_SMD:C_0603_1608Metric -> Capacitor_SMD:C_0805_2012Metric
- C38, C42: value 10pF, 10%, 10V -> 20pF, 10%, 10V
- C59: value 300nF, 10%, 50V -> 470nF, 10%, 50V; footprint Capacitor_SMD:C_0402_1005Metric -> Capacitor_SMD:C_0603_1608Metric
- L1: footprint Inductor_SMD:L_Coilcraft_XxL4040 -> Inductor_SMD:L_0603_1608Metric

Commit message: [Fix] Fix tcan4550 spi wrong connection
Signed-off-by: Homalozoa <nx.tardis@gmail.com>
Parts:
- removed TP4: SWDIO, TestPoint:TestPoint_Pad_D1.5mm, symbol Connector:TestPoint
- removed TP5: SWCLK, TestPoint:TestPoint_Pad_D1.5mm, symbol Connector:TestPoint
- added J2: gh1.25, 3p, Connector_JST:JST_GH_SM03B-GHS-TB_1x03-1MP_P1.25mm_Horizontal, symbol Connector:Conn_01x03_Female
Connections:
- net GND: now also J2.3 (Pin_3)
- net SWCLK: now also J2.2 (Pin_2)
- net SWDIO: now also J2.1 (Pin_1)
- net TCAN_SCK: now also U3.34 (PB13); no longer U3.35 (PB14)
- net TCAN_SCS: now also U3.33 (PB12); no longer U3.36 (PB15)
- net TCAN_SDI: now also U3.36 (PB15); no longer U3.33 (PB12)
- net TCAN_SDO: now also U3.35 (PB14); no longer U3.34 (PB13)
