File: flasher_esp/flasher_esp.kicad_pcb (KiCad board)
At the start: 2 copper layers, 0 parts

Commit message: [New] Complete PCB of flasher_esp
Signed-off-by: Homalozoa X <nx.tardis@gmail.com>
Parts:
- added C1: 0.1uf, Capacitor_SMD:C_0402_1005Metric, F.Cu at (102.6, 56.8)
- added C2: 4.7uf, Capacitor_SMD:C_0402_1005Metric, F.Cu at (102.6, 55.7)
- added C3: 1uf, Capacitor_SMD:C_0402_1005Metric, F.Cu at (100.7, 55.7)
- added C4: 100uf, Capacitor_SMD:C_0402_1005Metric, F.Cu at (100.7, 54.7)
- added C5: 4.7uf, Capacitor_SMD:C_0402_1005Metric, F.Cu at (105.3, 53.2)
- added C6: 0.1uf, Capacitor_SMD:C_0402_1005Metric, F.Cu at (105.3, 54.2)
- added D1: SP0503BAHT, Package_TO_SOT_SMD:SOT-143, B.Cu at (108.7, 60.2)
- added D2: MHT136UBCT, Capacitor_SMD:C_0402_1005Metric, F.Cu at (97.3, 61.2)
- added D3: NCD0402G1, Capacitor_SMD:C_0402_1005Metric, F.Cu at (97.3, 59.1)
- added D4: NCD0402W1, Capacitor_SMD:C_0402_1005Metric, F.Cu at (97.3, 64.4)
- added J1: TYPE-C-31-M-12, Rolling_Custom:HRO_TYPE-C-31-M-12, F.Cu at (110.5, 59.9)
- added J2: UART_NPWR, Connector_JST:JST_GH_BM03B-GHS-TBT_1x03-1MP_P1.25mm_Vertical, F.Cu at (90.0, 60.1)
- added J3: UART_FLASH_ESP, Connector_JST:JST_GH_BM05B-GHS-TBT_1x05-1MP_P1.25mm_Vertical, B.Cu at (90.0, 60.1)
- added R1: 47.5k, Resistor_SMD:R_0402_1005Metric, F.Cu at (102.6, 54.7)
- added R2: 22.1k, Resistor_SMD:R_0402_1005Metric, F.Cu at (102.6, 57.8)
- added R3: 1k, Resistor_SMD:R_0402_1005Metric, F.Cu at (101.1, 57.3)
- added R4: 200R, Resistor_SMD:R_0402_1005Metric, F.Cu at (96.3, 62.3)
- added R5: 200R, Resistor_SMD:R_0402_1005Metric, F.Cu at (96.3, 60.2)
- added R6: 200R, Resistor_SMD:R_0402_1005Metric, F.Cu at (96.3, 63.4)
- added REF**: TestPoint_Pad_D1.0mm, TestPoint:TestPoint_Pad_D1.0mm, F.Cu at (93.2, 53.4)
- added REF**: TestPoint_Pad_D1.0mm, TestPoint:TestPoint_Pad_D1.0mm, F.Cu at (108.4, 66.5)
- added REF**: TestPoint_Pad_D1.0mm, TestPoint:TestPoint_Pad_D1.0mm, B.Cu at (108.4, 66.5)
- added REF**: TestPoint_Pad_D1.0mm, TestPoint:TestPoint_Pad_D1.0mm, B.Cu at (93.2, 53.4)
- added U1: CP2102N-A02-GQFN24, Package_DFN_QFN:QFN-24-1EP_4x4mm_P0.5mm_EP2.6x2.6mm, F.Cu at (101.1, 61.1)
Routing:
- net GND: track 0.00 -> 84.6 mm
- net +3V3: track 0.00 -> 27.0 mm, vias 0 -> 2
- net +5V: track 0.00 -> 16.6 mm, vias 0 -> 1
- net RXD: track 0.00 -> 16.2 mm, vias 0 -> 2
- net TXD: track 0.00 -> 15.2 mm, vias 0 -> 2
- net DTR: track 0.00 -> 15.1 mm, vias 0 -> 1
- net RTS: track 0.00 -> 11.2 mm, vias 0 -> 1
- net Net-(C1-Pad1): track 0.00 -> 6.43 mm
- net D+: track 0.00 -> 5.91 mm, vias 0 -> 1
- net D-: track 0.00 -> 5.33 mm, vias 0 -> 1
- net TXT: track 0.00 -> 1.74 mm
- net RXT: track 0.00 -> 1.68 mm
- net Net-(U1-Pad9): track 0.00 -> 1.47 mm
- net Net-(D4-Pad2): track 0.00 -> 1.01 mm
- net Net-(D3-Pad2): track 0.00 -> 1.01 mm
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- added copper zone on F.Cu, net +3V3
- added copper zone on B.Cu, net GND
Other:
- board outline added: 27 x 16.7 mm
