File: cerebellum/cerebellum.kicad_sch (KiCad schematic)
At the start: 153 parts, among them J1 PWR_OUT, J2 PWR_IN, J3 Conn_01x04, J4 gh1.25, 3p, J5 CM4_A, J6 CM4_B, J7 RJ45, Q1 AP2300, U1 GD32F405VGHx, U2 TPS5430DDAR, U3 BMI088, U4 TCAN4550RGYRQ1, U5 ICP-20100, U6 TPS54231, U7 TCAN4550RGYRQ1, Y1 8M, Y2 40M, Y3 40M

Commit message: [New] Add USB ports to cerebellum
Signed-off-by: Homalozoa <nx.tardis@gmail.com>
Parts:
- added C? (x8): 100nF, 10%, 10V, Capacitor_SMD:C_0201_0603Metric, symbol Device:C
- added C?: 100nF, 10%, 10V, Capacitor_SMD:C_0402_1005Metric, symbol Device:C
- added J? (x4): USB_C_Receptacle, Rolling_Custom:USB_C_Receptacle_TYPE-C-324G-BCP24, symbol Connector:USB_C_Receptacle
- added J?: (no value), symbol Connector:USB_C_Receptacle_USB2.0
- added R?: 2.2k, Resistor_SMD:R_0201_0603Metric, symbol Device:R_US
- added R?: (no value), Resistor_SMD:R_0201_0603Metric, symbol Device:R_US
- added R?: 1M, Resistor_SMD:R_0402_1005Metric, symbol Device:R_US
- added U? (x5): TPD4EUSB30, Package_SON:USON-10_2.5x1.0mm_P0.5mm, symbol Power_Protection:TPD4EUSB30
- added U? (x4): ECMF04-4HSM10, Rolling_Custom:SON_4-4HSM10_STM, symbol Rolling_Custom:ECMF04-4HSM10
- added U? (x4): ECMF02-4CMX8, Rolling_Custom:MICRO_QFN-8L_STM, symbol Rolling_Custom:ECMF02-4CMX8
- added U?: (no value), symbol Power_Protection:TPD4EUSB30
- C? (x2): value (none) -> 22pF, 10%, 50V
- C? (x2): value (none) -> 100nF, 10%, 10V; footprint (none) -> Capacitor_SMD:C_0201_0603Metric
- J3: value Conn_01x04 -> (none)
- J4: value gh1.25, 3p -> (none)
- R?: value (none) -> 100k
- U?: value (none) -> APL3553; footprint (none) -> Package_TO_SOT_SMD:SOT-23-5
- U?: value (none) -> TPD4EUSB30
- U?: value (none) -> GD25Q40C
Connections:
- net +5V: now also J?.A4 (VBUS), J?.A4 (VBUS), J?.A4 (VBUS), J?.A4 (VBUS), J?.A4 (VBUS), J?.A9 (VBUS), J?.A9 (VBUS), J?.A9 (VBUS), J?.A9 (VBUS), J?.A9 (VBUS), J?.B4 (VBUS), J?.B4 (VBUS), J?.B4 (VBUS), J?.B4 (VBUS), J?.B4 (VBUS), J?.B9 (VBUS), J?.B9 (VBUS), J?.B9 (VBUS), J?.B9 (VBUS), J?.B9 (VBUS), R?.1, U?.1 (VBUS), U?.1 (VBUS), U?.1 (VBUS), U?.1 (VBUS)
- net GND: now also C?.1, J?.A1 (GND), J?.A1 (GND), J?.A1 (GND), J?.A1 (GND), J?.A1 (GND), J?.A12 (GND), J?.A12 (GND), J?.A12 (GND), J?.A12 (GND), J?.A12 (GND), J?.B1 (GND), J?.B1 (GND), J?.B1 (GND), J?.B1 (GND), J?.B1 (GND), J?.B12 (GND), J?.B12 (GND), J?.B12 (GND), J?.B12 (GND), J?.B12 (GND), R?.2, R?.2, U?.3 (GND), U?.3 (GND), U?.3 (GND), U?.3 (GND), U?.3 (GND), U?.3 (GND), U?.3 (GND), U?.3 (GND), U?.3 (GND), U?.3 (GND), U?.5 (GND), U?.5 (GND), U?.5 (GND), U?.5 (GND), U?.8 (GND), U?.8 (GND), U?.8 (GND), U?.8 (GND), U?.8 (GND), U?.8 (GND), U?.8 (GND), U?.8 (GND), U?.8 (GND), U?.8 (GND), U?.8 (GND), U?.8 (GND), U?.8 (GND), U?.8 (GND)
- net USB_N: now also J?.A7 (D-), J?.B7 (D-), U?.2 (D1-)
- net USB_OTG_ID: now also R?.1, R?.2
- net USB_P: now also J?.A6 (D+), J?.B6 (D+), U?.1 (D1+)
- net USB1_3TXP: now reaches U?.35 (U3TXDP1)
- net USB1_3TXP: now also C?.1
- net USB1_3TXN: now reaches U?.36 (U3TXDN1)
- net USB1_3TXN: now also C?.2
- net USB1_3RXP: now reaches U?.38 (U3RXDP1)
- net USB1_3RXP: now also U?.7 (D2+_IC)
- net USB1_3RXN: now reaches U?.39 (U3RXDN1)
- net USB1_3RXN: now also U?.6 (D2-_IC)
- net USB1_2P: now reaches U?.41 (U2DP1)
- net USB1_2P: now also U?.6 (D+_IC)
- net USB1_2N: now reaches U?.42 (U2DM1)
- net USB1_2N: now also U?.7 (D-_IC)
- net USB2_3TXP: now reaches U?.44 (U3TXDP2)
- net USB2_3TXP: now also C?.1
- net USB2_3TXN: now reaches U?.45 (U3TXDN2)
- net USB2_3TXN: now also C?.2
- net USB2_3RXP: now reaches U?.47 (U3RXDP2)
- net USB2_3RXP: now also U?.7 (D2+_IC)
- net USB2_3RXN: now reaches U?.48 (U3RXDN2)
- net USB2_2P: now reaches U?.50 (U2DP2)
- net USB2_2P: now also U?.6 (D+_IC)
- net USB2_2N: now reaches U?.51 (U2DM2)
- net USB2_2N: now also U?.7 (D-_IC)
- net USB3_3TXP: now reaches U?.52 (U3TXDP3)
- net USB3_3TXP: now also C?.1
- net USB3_3TXN: now reaches U?.53 (U3TXDN3)
- net USB3_3TXN: now also C?.2
- net USB3_3RXP: now reaches U?.55 (U3RXDP3)
- net USB3_3RXP: now also U?.7 (D2+_IC)
- net USB3_3RXN: now reaches U?.56 (U3RXDN3)
- net USB3_3RXN: now also U?.6 (D2-_IC)
- net USB3_2P: now reaches U?.58 (U2DP3)
- net USB3_2P: now also U?.6 (D+_IC)
- net USB3_2N: now reaches U?.59 (U2DM3)
- net USB3_2N: now also U?.7 (D-_IC)
- net USB4_3TXP: now reaches U?.61 (U3TXDP4)
- net USB4_3TXP: now also C?.1
- net USB4_3TXN: now reaches U?.62 (U3TXDN4)
- net USB4_3TXN: now also C?.2
- net USB4_3RXP: now reaches U?.64 (U3RXDP4)
- net USB4_3RXP: now also U?.7 (D2+_IC)
- net USB4_3RXN: now reaches U?.65 (U3RXDN4)
- net USB4_3RXN: now also U?.6 (D2-_IC)
- net USB4_2P: now reaches U?.67 (U2DP4)
- net USB4_2P: now also U?.6 (D+_IC)
- net USB4_2N: now reaches U?.68 (U2DM4)
- net USB4_2N: now also U?.7 (D-_IC)
- new net: C?.1, U?.9 (D1-_IC) (x4)
- new net: C?.2, U?.10 (D1+_IC) (x4)
- new net Con_USB1_2N: J?.A7 (D-), J?.B7 (D-), U?.2 (D1-), U?.3 (D+_Con)
- new net Con_USB1_2P: J?.A6 (D+), J?.B6 (D+), U?.1 (D1+), U?.2 (D-_Con)
- new net Con_USB1_3RXN: J?.A10 (RX2-), J?.B10 (RX1-), U?.2 (D1-), U?.2 (D1-), U?.2 (D1-), U?.5 (D2-_Con)
- new net Con_USB1_3RXP: J?.A11 (RX2+), J?.B11 (RX1+), U?.1 (D1+), U?.1 (D1+), U?.1 (D1+), U?.4 (D2+_Con)
- new net Con_USB1_3TXN: J?.A3 (TX1-), J?.B3 (TX2-), U?.2 (D1-_Con), U?.5 (D2-), U?.5 (D2-), U?.5 (D2-)
- new net Con_USB1_3TXP: J?.A2 (TX1+), J?.B2 (TX2+), U?.1 (D1+_Con), U?.4 (D2+), U?.4 (D2+), U?.4 (D2+)
- new net Con_USB2_2N: J?.A7 (D-), J?.B7 (D-), U?.3 (D+_Con), U?.5 (D2-)
- new net Con_USB2_2P: J?.A6 (D+), J?.B6 (D+), U?.2 (D-_Con), U?.4 (D2+)
- new net Con_USB2_3RXN: J?.A10 (RX2-), J?.B10 (RX1-), U?.5 (D2-_Con)
- new net Con_USB2_3RXP: J?.A11 (RX2+), J?.B11 (RX1+), U?.4 (D2+_Con)
- new net Con_USB2_3TXN: J?.A3 (TX1-), J?.B3 (TX2-), U?.2 (D1-_Con)
- new net Con_USB2_3TXP: J?.A2 (TX1+), J?.B2 (TX2+), U?.1 (D1+_Con)
- new net Con_USB3_2N: J?.A7 (D-), J?.B7 (D-), U?.2 (D1-), U?.3 (D+_Con)
- new net Con_USB3_2P: J?.A6 (D+), J?.B6 (D+), U?.1 (D1+), U?.2 (D-_Con)
- new net Con_USB3_3RXN: J?.A10 (RX2-), J?.B10 (RX1-), U?.5 (D2-_Con)
- new net Con_USB3_3RXP: J?.A11 (RX2+), J?.B11 (RX1+), U?.4 (D2+_Con)
- new net Con_USB3_3TXN: J?.A3 (TX1-), J?.B3 (TX2-), U?.2 (D1-_Con)
- new net Con_USB3_3TXP: J?.A2 (TX1+), J?.B2 (TX2+), U?.1 (D1+_Con)
- new net Con_USB4_2N: J?.A7 (D-), J?.B7 (D-), U?.3 (D+_Con), U?.5 (D2-)
- new net Con_USB4_2P: J?.A6 (D+), J?.B6 (D+), U?.2 (D-_Con), U?.4 (D2+)
- new net Con_USB4_3RXN: J?.A10 (RX2-), J?.B10 (RX1-), U?.5 (D2-_Con)
- new net Con_USB4_3RXP: J?.A11 (RX2+), J?.B11 (RX1+), U?.4 (D2+_Con)
- new net Con_USB4_3TXN: J?.A3 (TX1-), J?.B3 (TX2-), U?.2 (D1-_Con)
- new net Con_USB4_3TXP: J?.A2 (TX1+), J?.B2 (TX2+), U?.1 (D1+_Con)
- new net GNDPWR: C?.2, J?.S1 (SHIELD), J?.S1 (SHIELD), J?.S1 (SHIELD), J?.S1 (SHIELD), J?.S1 (SHIELD), R?.1
- no-connect marks 166 -> 169
Other:
- note removed: "Connectors"
- moved on the sheet: C13, C17, C19, C21, C24, C28, C33, C34, C35, C36, C37, C38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
